File: Schematic/Mainboard/Mainboard.kicad_sch (KiCad schematic)
At the start: 18 parts, among them J1 Motor_A, J2 Motor_B, J3 Motor_C, J4 BATT_IN, J5 Servo, J6 Servo, J7 ESC, J8 ESC_PWR, SW1 MAIN_CUTOFF, U4 RFM69HW, U5 XL60019_Boost_Module, U6 Mini360

Commit message: set up radio module on ESP32
also worked on getting the ESP32 debugger up and running
Connections:
- net ESC: now also U?.24 (D4); no longer U?.25 (RX2/D16)
- net M A1: now also U?.25 (RX2/D16); no longer U?.27 (TX2/D17)
- net M A2: now also U?.27 (TX2/D17); no longer U?.34 (D5)
- net M B1: now also U?.35 (D18); no longer U?.36 (D23)
- net M B2: now also U?.34 (D5); no longer U?.35 (D18)
- net SERVO 1: now also U?.22 (D2); no longer U?.23 (D0)
- net SERVO 2: now also U?.23 (D0); no longer U?.24 (D4)
- net +12V renamed +10V
- net +10V: no longer U2.1 (SLEEP), U3.1 (SLEEP)
- new net SLEEP: U2.1 (SLEEP), U3.1 (SLEEP), U?.36 (D23)
- no-connect marks 20 -> 19
Changed lines of the file:
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@@
   (no_connect (at 83.82 57.15))
   (no_connect (at 52.07 39.37))
-  (no_connect (at 83.82 54.61))
   (no_connect (at 144.78 46.99))
   (no_connect (at 52.07 34.29))
@@
     (effects (font (size 1.27 1.27)) (justify right bottom))
   )
-  (label "M A2" (at 83.82 41.91 0) (fields_autoplaced)
+  (label "M A2" (at 83.82 44.45 0) (fields_autoplaced)
     (effects (font (size 1.27 1.27)) (justify left bottom))
   )
@@
     (effects (font (size 1.27 1.27)) (justify right bottom))
   )
-  (label "SERVO 1" (at 83.82 52.07 0) (fields_autoplaced)
+  (label "SERVO 1" (at 83.82 54.61 0) (fields_autoplaced)
     (effects (font (size 1.27 1.27)) (justify left bottom))
   )
@@
     (effects (font (size 1.27 1.27)) (justify right bottom))
   )
-  (label "M B1" (at 83.82 36.83 0) (fields_autoplaced)
+  (label "M B1" (at 83.82 39.37 0) (fields_autoplaced)
     (effects (font (size 1.27 1.27)) (justify left bottom))
   )
@@
     (effects (font (size 1.27 1.27)) (justify right bottom))
   )
-  (label "SERVO 2" (at 83.82 49.53 0) (fields_autoplaced)
-    (effects (font (size 1.27 1.27)) (justify left bottom))
-  )
-  (label "ESC" (at 83.82 46.99 0) (fields_autoplaced)
+  (label "SERVO 2" (at 83.82 52.07 0) (fields_autoplaced)
+    (effects (font (size 1.27 1.27)) (justify left bottom))
+  )
+  (label "SLEEP" (at 124.46 31.75 180) (fields_autoplaced)
+    (effects (font (size 1.27 1.27)) (justify right bottom))
+  )
+  (label "ESC" (at 83.82 49.53 0) (fields_autoplaced)
     (effects (font (size 1.27 1.27)) (justify left bottom))
   )
@@
     (effects (font (size 1.27 1.27)) (justify right bottom))
   )
+  (label "SLEEP" (at 83.82 36.83 0) (fields_autoplaced)
+    (effects (font (size 1.27 1.27)) (justify left bottom))
+  )
+  (label "SLEEP" (at 124.46 55.88 180) (fields_autoplaced)
+    (effects (font (size 1.27 1.27)) (justify right bottom))
+  )
   (label "AUX" (at 198.12 74.93 0) (fields_autoplaced)
     (effects (font (size 1.27 1.27)) (justify left bottom))
@@
     (effects (font (size 1.27 1.27)) (justify right bottom))
   )
-  (label "M B2" (at 83.82 39.37 0) (fields_autoplaced)
+  (label "M B2" (at 83.82 41.91 0) (fields_autoplaced)
     (effects (font (size 1.27 1.27)) (justify left bottom))
   )
@@
     (effects (font (size 1.27 1.27)) (justify left bottom))
   )
-  (label "M A1" (at 83.82 44.45 0) (fields_autoplaced)
+  (label "M A1" (at 83.82 46.99 0) (fields_autoplaced)
     (effects (font (size 1.27 1.27)) (justify left bottom))
   )
@@
         (path "/dc068368-f26a-439a-bd25-832d8f26a4bd"
           (reference "#FLG04") (unit 1)
-        )
-      )
-    )
-  )
-  (symbol (lib_id "power:+12V") (at 144.78 41.91 270) (unit 1)
-    (in_bom yes) (on_board yes) (dnp no) (fields_autoplaced)
-    (property "Reference" "#PWR06" (at 140.97 41.91 0)
-      (effects (font (size 1.27 1.27)) hide)
-    )
-    (property "Value" "+12V" (at 148.59 41.91 90)
-      (effects (font (size 1.27 1.27)) (justify left))
-    )
-    (property "Footprint" "" (at 144.78 41.91 0)
-      (effects (font (size 1.27 1.27)) hide)
-    )
-    (property "Datasheet" "" (at 144.78 41.91 0)
-      (effects (font (size 1.27 1.27)) hide)
-    )
-    (pin "1")
-    (instances
-      (project "Mainboard"
-        (path "/dc068368-f26a-439a-bd25-832d8f26a4bd"
-          (reference "#PWR06") (unit 1)
         )
       )
@@
     )
   )
-  (symbol (lib_id "power:+12V") (at 215.9 27.94 0) (unit 1)
-    (in_bom yes) (on_board yes) (dnp no) (fields_autoplaced)
-    (property "Reference" "#PWR015" (at 215.9 31.75 0)
-      (effects (font (size 1.27 1.27)) hide)
-    )
-    (property "Value" "+12V" (at 215.9 22.86 0)
-      (effects (font (size 1.27 1.27)))
-    )
-    (property "Footprint" "" (at 215.9 27.94 0)
-      (effects (font (size 1.27 1.27)) hide)
-    )
-    (property "Datasheet" "" (at 215.9 27.94 0)
-      (effects (font (size 1.27 1.27)) hide)
-    )
-    (pin "1")
-    (instances
-      (project "Mainboard"
-        (path "/dc068368-f26a-439a-bd25-832d8f26a4bd"
-          (reference "#PWR015") (unit 1)
-        )
-      )
-    )
-  )
   (symbol (lib_id "Connector_Generic:Conn_01x03") (at 233.68 57.15 0) (unit 1)
     (in_bom yes) (on_board yes) (dnp no) (fields_autoplaced)
@@
         (path "/dc068368-f26a-439a-bd25-832d8f26a4bd"
           (reference "J2") (unit 1)
+        )
+      )
+    )
+  )
+  (symbol (lib_id "power:+10V") (at 144.78 66.04 270) (unit 1)
+    (in_bom yes) (on_board yes) (dnp no) (fields_autoplaced)
+    (property "Reference" "#PWR08" (at 140.97 66.04 0)
+      (effects (font (size 1.27 1.27)) hide)
+    )
+    (property "Value" "+10V" (at 148.59 66.04 90)
+      (effects (font (size 1.27 1.27)) (justify left))
+    )
+    (property "Footprint" "" (at 144.78 66.04 0)
+      (effects (font (size 1.27 1.27)) hide)
+    )
+    (property "Datasheet" "" (at 144.78 66.04 0)
+      (effects (font (size 1.27 1.27)) hide)
+    )
+    (pin "1")
+    (instances
+      (project "Mainboard"
+        (path "/dc068368-f26a-439a-bd25-832d8f26a4bd"
+          (reference "#PWR08") (unit 1)
         )
       )
@@
     )
   )
-  (symbol (lib_id "power:+12V") (at 124.46 55.88 0) (unit 1)
-    (in_bom yes) (on_board yes) (dnp no) (fields_autoplaced)
-    (property "Reference" "#PWR04" (at 124.46 59.69 0)
-      (effects (font (size 1.27 1.27)) hide)
-    )
-    (property "Value" "+12V" (at 124.46 50.8 0)
-      (effects (font (size 1.27 1.27)))
-    )
-    (property "Footprint" "" (at 124.46 55.88 0)
-      (effects (font (size 1.27 1.27)) hide)
-    )
-    (property "Datasheet" "" (at 124.46 55.88 0)
-      (effects (font (size 1.27 1.27)) hide)
-    )
-    (pin "1")
-    (instances
-      (project "Mainboard"
-        (path "/dc068368-f26a-439a-bd25-832d8f26a4bd"
-          (reference "#PWR04") (unit 1)
-        )
-      )
-    )
-  )
   (symbol (lib_id "power:+BATT") (at 152.4 116.84 180) (unit 1)
     (in_bom yes) (on_board yes) (dnp no) (fields_autoplaced)
@@
         (path "/dc068368-f26a-439a-bd25-832d8f26a4bd"
           (reference "#PWR018") (unit 1)
-        )
-      )
-    )
-  )
-  (symbol (lib_id "power:+12V") (at 124.46 31.75 0) (unit 1)
-    (in_bom yes) (on_board yes) (dnp no) (fields_autoplaced)
-    (property "Reference" "#PWR03" (at 124.46 35.56 0)
-      (effects (font (size 1.27 1.27)) hide)
-    )
-    (property "Value" "+12V" (at 124.46 26.67 0)
-      (effects (font (size 1.27 1.27)))
-    )
-    (property "Footprint" "" (at 124.46 31.75 0)
-      (effects (font (size 1.27 1.27)) hide)
-    )
-    (property "Datasheet" "" (at 124.46 31.75 0)
-      (effects (font (size 1.27 1.27)) hide)
-    )
-    (pin "1")
-    (instances
-      (project "Mainboard"
-        (path "/dc068368-f26a-439a-bd25-832d8f26a4bd"
-          (reference "#PWR03") (unit 1)
         )
       )
@@
     )
   )
+  (symbol (lib_id "power:+10V") (at 144.78 41.91 270) (unit 1)
+    (in_bom yes) (on_board yes) (dnp no) (fields_autoplaced)
+    (property "Reference" "#PWR06" (at 140.97 41.91 0)
+      (effects (font (size 1.27 1.27)) hide)
+    )
+    (property "Value" "+10V" (at 148.59 41.91 90)
+      (effects (font (size 1.27 1.27)) (justify left))
+    )
+    (property "Footprint" "" (at 144.78 41.91 0)
+      (effects (font (size 1.27 1.27)) hide)
+    )
+    (property "Datasheet" "" (at 144.78 41.91 0)
+      (effects (font (size 1.27 1.27)) hide)
+    )
+    (pin "1")
+    (instances
+      (project "Mainboard"
+        (path "/dc068368-f26a-439a-bd25-832d8f26a4bd"
+          (reference "#PWR06") (unit 1)
+        )
+      )
+    )
+  )
   (symbol (lib_id "Connector_Generic:Conn_01x02") (at 113.03 60.96 180) (unit 1)
     (in_bom yes) (on_board yes) (dnp no)
@@
         (path "/dc068368-f26a-439a-bd25-832d8f26a4bd"
           (reference "J1") (unit 1)
-        )
-      )
-    )
-  )
-  (symbol (lib_id "power:+12V") (at 144.78 66.04 270) (unit 1)
-    (in_bom yes) (on_board yes) (dnp no) (fields_autoplaced)
-    (property "Reference" "#PWR08" (at 140.97 66.04 0)
-      (effects (font (size 1.27 1.27)) hide)
-    )
-    (property "Value" "+12V" (at 148.59 66.04 90)
-      (effects (font (size 1.27 1.27)) (justify left))
-    )
-    (property "Footprint" "" (at 144.78 66.04 0)
-      (effects (font (size 1.27 1.27)) hide)
-    )
-    (property "Datasheet" "" (at 144.78 66.04 0)
-      (effects (font (size 1.27 1.27)) hide)
-    )
-    (pin "1")
-    (instances
-      (project "Mainboard"
-        (path "/dc068368-f26a-439a-bd25-832d8f26a4bd"
-          (reference "#PWR08") (unit 1)
         )
       )
@@
         )
       )
+    )
+  )
+  (symbol (lib_id "power:+10V") (at 215.9 27.94 0) (unit 1)
+    (in_bom yes) (on_board yes) (dnp no) (fields_autoplaced)
+    (property "Reference" "#PWR015" (at 215.9 31.75 0)
+      (effects (font (size 1.27 1.27)) hide)
+    )
+    (property "Value" "+10V" (at 215.9 22.86 0)
+      (effects (font (size 1.27 1.27)))
+    )
+    (property "Footprint" "" (at 215.9 27.94 0)
+      (effects (font (size 1.27 1.27)) hide)
+    )
+    (property "Datasheet" "" (at 215.9 27.94 0)
+      (effects (font (size 1.27 1.27)) hide)
+    )
+    (pin "1")
+    (instances
+      (project "Mainboard"
+        (path "/dc068368-f26a-439a-bd25-832d8f26a4bd"
+          (reference "#PWR015") (unit 1)
+        )
+      )

Commit message: Work on weight reduction
thin the shell in order to get the total weight under 1 lb.
Parts:
- added R2: 150k Ohm, Resistor_THT:R_Axial_DIN0207_L6.3mm_D2.5mm_P7.62mm_Horizontal, symbol Device:R
- added R3: 10k Ohm, Resistor_THT:R_Axial_DIN0207_L6.3mm_D2.5mm_P7.62mm_Horizontal, symbol Device:R
- renumbered J8 to J10, J1 to J3, J2 to J4, J3 to J5, J4 to J6, J5 to J7, J6 to J8, J7 to J9
Connections:
- net +BATT SW: now also R2.2
- net GND: now also R3.1
- net INTER: now also U?.11 (D35); no longer U?.17 (D14)
- net BAT READ: now reaches U?.10 (D34)
- net BAT READ: now also R2.1, R3.2
- net TCK: now reaches U?.20 (D13)
- net TDO: now reaches U?.21 (D15)
- net AUX: no longer names the net of U4.6 (DIO4)
- net AUX: no longer U?.18 (D12)
- new net TDI: U?.18 (D12)
- new net TMS: U?.17 (D14)
- no-connect marks 19 -> 16
Other:
- note added: "Voltmeter Assembly"

Commit message: prepare to mill PCB
also add more sub-functions to firmware
Parts:
- renumbered J3 to J1, J4 to J2, J5 to J3, J6 to J4, J7 to J5, J8 to J6, J9 to J7, J10 to J8
Other:
- moved on the sheet: R2, R3
