File: RB3/Schematic/Schematic/Schematic.kicad_sch (KiCad schematic)
At the start: 9 parts, among them J1 Motor 1, J2 Motor 2, J3 Battery, J7 ESC, J8 ESC_PWR, SW1 MAIN_CUTOFF, U3 Mini360

Commit message: lots of CAD and firmware work
back to basics: re-establish communication between two ESP32s because that was broken in the higher-level code.
Parts:
- J1: footprint (none) -> Connector_PinHeader_2.54mm:PinHeader_1x06_P2.54mm_Vertical
- J2: value Motor 2 -> Motor 1; footprint (none) -> Connector_PinHeader_2.54mm:PinHeader_1x06_P2.54mm_Vertical
- J3: footprint (none) -> Connector_PinHeader_2.54mm:PinHeader_1x02_P2.54mm_Vertical
Connections:
- net +3.3V: now also J1.2 (Pin_2), J2.2 (Pin_2), U1.14 (3v3); no longer J1.E+ (Pin_2), J2.E+ (Pin_2), U1.3 (3v3)
- net ESC: now also U1.1 (D5); no longer U1.16 (D5)
- net GND: now also J1.5 (Pin_5), J2.5 (Pin_5), U1.15 (Gnd); no longer J1.EG (Pin_5), J2.EG (Pin_5), U1.2 (Gnd)
- net M1 A: now also J1.1 (Motor_2); no longer J1.M2 (Motor_2)
- net M1 B: now also J1.6 (M1); no longer J1.M1
- net M1 Control A: now also U1.9 (D0); no longer U1.5 (D3)
- net M1 Control B: now also U1.10 (D1); no longer U1.6 (D2)
- net M1 EA: now also J1.4 (Pin_4), U1.5 (D9); no longer J1.EA (Pin_4), U1.15 (D6)
- net M1 EB: now also J1.3 (Pin_3), U1.4 (D8); no longer J1.EB (Pin_3), U1.14 (D7)
- net M2 A: now also J2.1 (Motor_2); no longer J2.M2 (Motor_2)
- net M2 B: now also J2.6 (M1); no longer J2.M1
- net M2 Control A: now also U1.11 (D2); no longer U1.7 (D1)
- net M2 Control B: now also U1.12 (D3); no longer U1.8 (D0)
- net M2 EA: now also J2.4 (Pin_4), U1.3 (D7); no longer J2.EA (Pin_4), U1.13 (D8)
- net M2 EB: now also J2.3 (Pin_3), U1.2 (D6); no longer J2.EB (Pin_3), U1.12 (D9)
- net SLEEP: now also U1.13 (D4); no longer U1.4 (D4)
Other:
- note added: "M1 - WHITE GND - BLUE C1 - GREEN C2 - YELLOW VCC - BLACK M2 - RED"
- moved on the sheet: U1
