File: RB4/Schematic/LOLIN32 pinLabels_RFM.kicad_sch (KiCad schematic)
At the start: 2 parts, among them U1 ESP32-LOLIN32-Lite

Commit message: Finish the thing before competition day
This robot is cursed
Parts:
- added U2: RFM69HW, RF_Module:HOPERF_RFM69HW, symbol My_Library:RFM69HW
Connections:
- net Battery Reader is gone; now on net Input only, no internal pullups: U1.10 (D34)
- net Buzzer is gone; now on net Can't Pull HIGH at boot, out good: U1.18 (D12)
- net ESC Left is gone; now on net GOOD: U1.35 (D18)
- net ESC Right is gone; now on net GOOD: U1.36 (D23)
- net Encoder A is gone; now on net Out Good, (floating or LOW to flash): U1.22 (D2)
- net Encoder B is gone; now on net PWM at boot: U1.21 (D15)
- net Encoder Switch is gone; now on net GOOD: U1.20 (D13)
- net FireTrg is gone; now on net OK, PWM at boot: U1.34 (D5)
- net IR Emitter is gone; now on net GOOD: U1.13 (D33)
- net IR Rec. Supply is gone; now on net GOOD: U1.12 (D32)
- net IR Reciever is gone; now on net Input only, no internal pullups: U1.11 (D35)
- net MagTrg is gone; now on net GOOD (Pin 17): U1.27 (TX2/D17)
- net Preset A is gone; now on net PWM at boot: U1.17 (D14)
- net Preset B is gone; now on net GOOD: U1.16 (D27)
- net Preset C is gone; now on net GOOD: U1.15 (D26)
- net Pusher Pin is gone; now on net GOOD: U1.14 (D25)
- net SCL/SCK (Clock) is gone; now on net GOOD: U1.39 (D22)
- net SDA/SDI (Data) is gone; now on net GOOD: U1.38 (D19)
- net SolenoidTrig A is gone; now on net GOOD: U1.24 (D4)
- net SolenoidTrig B is gone; now on net PWM at boot, pulled up input only (LOW to flash): U1.23 (D0)
- net +3V3: no longer names the net of U1.40 (3V3)
- net GND: no longer names the net of U1.19 (GND)
- net RevTrg renamed RADIO INPUT
- new net 18: U2.12 (SCK)
- new net 19: U2.14 (MOSI)
- new net 22: U2.15 (NSS)
- new net 23: U2.13 (MISO)
- new net D32: U2.1 (RESET)
- new net D33: U2.2 (DIO0)
