File: RB4/Schematic/Schematic/Schematic.kicad_sch (KiCad schematic)
At the start: 9 parts, among them J1 Battery, J2 Motor 1, J3 Motor 2, J4 ESC, SW1 MAIN_CUTOFF, U1 RFM69HW, U3 LD1117V33

Commit message: Lots of work on RB4
so much to do in so little time
Parts:
- added U5, U6: ~, Espressif:ESP32-C3-SuperMini_PLUS, symbol Espressif:ESP32-C3-SuperMini_PLUS
- added U7: RFM69HW, RF_Module:HOPERF_RFM69HW, symbol My_Library:RFM69HW
Connections:
- net +3.3V: now also U6.14 (3v3), U7.8 (3.3V)
- net GND: now also U6.15 (Gnd), U7.9 (GND)
- net INTER: now also U6.3 (D7), U7.2 (DIO0)
- net M1 Control A: now also U6.5 (D9)
- net M1 Control B: now also U6.4 (D8)
- net M2 Control A: now also U6.2 (D6)
- net M2 Control B: now also U6.1 (D5)
- net MISO: now also U6.11 (D2), U7.13 (MISO)
- net MOSI: now also U6.10 (D1), U7.14 (MOSI)
- net NSS: now also U6.9 (D0), U7.15 (NSS)
- net RESET: now also U6.6 (D10), U7.1 (RESET)
- net SCK: now also U6.12 (D3)
- net SLEEP: now also U6.13 (D4)
- new net BOOT, OUT GOOD: U5.5 (D9)
- new net GOOD: U5.1 (D5), U5.10 (D1), U5.12 (D3), U5.13 (D4), U5.2 (D6), U5.3 (D7), U5.6 (D10), U5.9 (D0)
- new net HIGH IN ON START, OUT GOOD: U5.11 (D2), U5.4 (D8)
- new net USED FOR PRINT: U5.7 (D20/RX), U5.8 (D21/TX)
- no-connect marks 10 -> 12

Commit message: Finish the thing before competition day
This robot is cursed
Parts:
- added U8: ~, My_Library:HW-627, symbol My_Library:HW-627
- added U9: ~, Espressif:ESP32-C3-SuperMini_PLUS, symbol Espressif:ESP32-C3-SuperMini_PLUS
Connections:
- net GOOD: now also U9.10 (D1), U9.12 (D3), U9.13 (D4), U9.9 (D0)
- net HIGH IN ON START, OUT GOOD: now also U9.11 (D2); no longer U5.4 (D8)
- net USED FOR PRINT: now also U9.7 (D20/RX), U9.8 (D21/TX)
- new net: U8.12 (IN4), U9.1 (D5)
- new net: U8.11 (IN3), U9.2 (D6)
- new net: U8.8 (IN2), U9.5 (D9)
- new net: U8.7 (IN1), U9.6 (D10)
- new net HIGH IN ON START, OUT GOOD, LED: U5.4 (D8)
- no-connect marks 12 -> 13
Other:
- moved on the sheet: U5
